File: schematics/tipi-interface.sch (KiCad schematic (older format))
At the start: 17 parts

Commit message: Update schematic to separate input from output.
Separate gpio pins will be used on RPi. This should prevent needing to switch GPIO pin modes frequently, as well as disable reading what is output. Write port is 0x5FFF, read port is 0x5FEF.

Still needs flow control signals, and a CRU enable bit.
Parts:
- removed R2: 1k, symbol R
- removed U?: 74HC245, symbol 74HC245
- removed U?: 74HC04, symbol 74HC04
- removed U?: 7400, symbol 7400
- added R3, R?: 1k, symbol R
- added U?: 74LVC245, symbol 74LVC245
- added U?: 74LS20, symbol 74LS20
- added U?: 74HC04, symbol 74HC04
Connections:
- net labels added: CRUCLK*, GPIO33, GPIO34, GPIO35, GPIO36, GPIO37, GPIO38, GPIO39, GPIO7, MEMEN*, WE*
- net labels removed: CRUCLK, MEMEN, WE
- wire segments 130 -> 146
Other:
- moved on the sheet: U?
