File: xc9500-schematic/smd-tipi-interface.sch (KiCad schematic (older format))
At the start: 24 parts

Commit message: fix dsr rom address maping in schematic
Parts:
- D? (x9): symbol LED -> LED-RESCUE-smd-tipi-interface
Connections:
- net A0: no longer U?.27 (A14)
- net A1: no longer U?.26 (A13)
- net A10: now also U?.5 (A5); no longer U?.6 (A4)
- net A11: now also U?.6 (A4); no longer U?.7 (A3)
- net A12: now also U?.7 (A3); no longer U?.8 (A2)
- net A13: now also U?.8 (A2)
- net A14: now also U?.9 (A1)
- net A15: now also U?.10 (A0)
- net A2: no longer U?.2 (A12)
- net A3: now also U?.2 (A12); no longer U?.23 (A11)
- net A4: now also U?.23 (A11); no longer U?.21 (A10)
- net A5: now also U?.21 (A10); no longer U?.24 (A9)
- net A6: now also U?.24 (A9); no longer U?.25 (A8)
- net A7: now also U?.25 (A8); no longer U?.3 (A7)
- net A8: now also U?.3 (A7); no longer U?.4 (A6)
- net A9: now also U?.4 (A6); no longer U?.5 (A5)
- net at U?.10 (P10): now also U?.26 (A13); no longer U?.10 (A0)
- net at U?.9 (P9): now also U?.27 (A14); no longer U?.9 (A1)
