File: tipi-peb-kicad/tipi-peb.sch (KiCad schematic (older format))
At the start: 32 parts, among them Q1 Q_NPN_BCE, T1 TEST_1P, T2 TEST_1P, T3 TEST_1P, T4 TEST_1P, T5 TEST_1P, U1 XC95144XL-TQ100, U2 27C256, U3 74HCT245, U4 LM1117-3.3

Commit message: kicad work on peb card, added buffers, and ama-d decoding
Parts:
- added C? (x4): 0.1uf, Capacitors_SMD:C_0805_HandSoldering, symbol C_Small
- added R7, R8, R?: 1k, Resistors_SMD:R_0805_HandSoldering, symbol R
- added U5: 74LS138, symbol 74LS138
- added U6, U7, U8: 74HC244, symbol 74HC244
- CRUBASE1: symbol CONN_02X04 -> Conn_02x04_Counter_Clockwise
- RPi1: symbol CONN_02X05 -> Conn_02x05_Counter_Clockwise
Connections:
- net labels added: TI-AMD, TI_A0, TI_A1, TI_A10, TI_A11, TI_A12, TI_A13, TI_A14, TI_A15, TI_A2, TI_A3, TI_A4, TI_A5, TI_A6, TI_A7, TI_A8, TI_A9, TI_AMA, TI_AMB, TI_AMC, TI_AME, TI_CRUCLK, TI_CRUIN, TI_DBIN, TI_MEMEN, TI_PH3, TI_WE
- net labels removed: B_CRUIN, B_EXTINT
- wire segments 53 -> 72
Other:
- moved on the sheet: C1, C10, C11, C2, C3, C4, C5, C6, C7, C8, C9, D1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

Commit message: working on peb schematic
Parts:
- added C15: 10uf, Capacitors_SMD:C_0805_HandSoldering, symbol CP1_Small
- added C17: 22uf, Capacitors_SMD:C_0805_HandSoldering, symbol CP1_Small
- added U9: LM7805_TO220, TO_SOT_Packages_THT:TO-220_Vertical, symbol LM7805_TO220
- gave numbers to parts that had none: 5
- renumbered C7 to C10, C8 to C11, C9 to C12, C10 to C13, C1 to C14, C2 to C16, C11 to C2, C3 to C5, C4 to C6, C5 to C7, C6 to C9, R7 to R2, R8 to R3, R3 to R4, R1 to R5, R2 to R6, R4 to R7, R5 to R8, R6 to R9, T5 to T1, T4 to T2, T2 to T4, T1 to T5, U5 to U1, U6 to U3, U7 to U4, U8 to U5, U1 to U6, U3 to U7, U4 to U8
Connections:
- net +5V: now also C17.1, U9.3 (VO); no longer C14.1, U8.3 (VI)
- net B_MEMEN: now also U6.99 (I/O/GSR)
- net GND: now also E1.20 (GND), E1.27 (GND), E1.3 (GND), E1.47 (GND), E1.49 (GND), E1.5 (GND), E1.53 (GND), E1.7 (GND), C15.2, C17.2, U9.2 (GND)
- net +8V: now reaches E1.1 (+8v)
- net +8V: now also C14.1, U8.3 (VI), C15.1, U9.1 (VI)
- no-connect marks 3 -> 65
Other:
- moved on the sheet: C14, C16, CRUBASE1, D1, E1, Q1, R4, R5, R6, U8

Commit message: edge card component
Parts:
- added R10, R11: 4.7k, Resistors_SMD:R_0805_HandSoldering, symbol R
- E1: footprint (none) -> peb-edge-card:ti99-peb-edge
- U1: value 74LS138 -> 74HCT138; footprint (none) -> SMD_Packages:SO-16-W
- U3, U4, U5: value 74HC244 -> 74HCT244; footprint (none) -> SMD_Packages:SSOP-20
- U9: footprint TO_SOT_Packages_THT:TO-220_Vertical -> TO_SOT_Packages_SMD:SOT-223
Connections:
- net TI_MEMEN is gone; now on net TI_AMD: E1.56 (MEMEN*), U1.4 (E1)
- net +5V: now also R10.2
- net DB_EN: now also U3.19 (2OE)
- net GND: now also R11.2
- net TI_AME: now also U1.6 (E3), R10.1; no longer U1.5 (E2)
- net RDBENA: now reaches E1.11 (RDBENA*)
- net RDBENA: now also U3.9 (2Y3)
- net at R1.2, U3.1 (1OE): now also U3.11 (2A3)
- net TI-AMD renamed TI_AMD
- net TI_AMD: now also U1.5 (E2), R11.1; no longer U1.6 (E3)
- no-connect marks 65 -> 61
