File: hardware/tipi-sideport/kicad/tipi.sch (KiCad schematic (older format))
At the start: 32 parts, among them J1 TI32kSideport, Q1 Q_NPN_BCE, T1 TEST_1P, T2 TEST_1P, T3 TEST_1P, T4 TEST_1P, T5 TEST_1P, U1 XC95144XL-TQ100, U2 27C256, U3 74HCT245, U4 LM1117-3.3

Commit message: results of loading in new version of kicad
Parts:
- C1, C2: symbol CP1_Small -> tipi-rescue:CP1_Small
- C10, C11, C3, C4, C5, C6, C7, C8, C9: symbol C_Small -> tipi-rescue:C_Small
- CRUBASE1: symbol CONN_02X04 -> tipi-rescue:CONN_02X04
- D1: symbol LED_ALT -> tipi-rescue:LED_ALT
- J1: symbol TI32kSideport -> ti32ksideport:TI32kSideport
- JTAG1: symbol AVR-JTAG-10 -> tipi-rescue:AVR-JTAG-10
- Q1: symbol Q_NPN_BCE -> tipi-rescue:Q_NPN_BCE
- R1, R2, R3: symbol R -> tipi-rescue:R
- R4, R5, R6: symbol R_Small -> tipi-rescue:R_Small
- RPi1: symbol CONN_02X05 -> tipi-rescue:CONN_02X05
- T1, T2, T3, T4, T5: symbol TEST_1P -> tipi-rescue:TEST_1P
- U1: symbol XC95144XL-TQ100 -> tipi-rescue:XC95144XL-TQ100
- U2: symbol 27C256 -> tipi-rescue:27C256
- U3: symbol 74LS245 -> tipi-rescue:74LS245
- U4: symbol LM1117-3.3-RESCUE-tipi -> tipi-rescue:LM1117-3.3-RESCUE-tipi
