File: hardware/tipi-speech/kicad/VS-Tipi.sch (KiCad schematic (older format))
At the start: 32 parts, among them J1 TI-99_Sideport, J2 USB_B_Micro, P1 TI-99_Sideport, Q1 NPN_BCE, U1 XC95144XL-TQ100, U2 27C256, U3 74HCT245, U4 LM1117-3.3, U5 CY62256L-70PC

Commit message: TIPI-32K V1 HW and CPLD update
V1 hardware and CPLD updates to add power tap and make RAM disableable.
Parts:
- added J3: Conn_01x02, Connector_PinHeader_2.54mm:PinHeader_1x02_P2.54mm_Horizontal, symbol Connector_Generic:Conn_01x02
- C1: LCSC (none) -> C15850
- C12, C3, C6: LCSC (none) -> C49678
- C2: LCSC (none) -> C45783
- J2: footprint Connector_USB:USB_Micro-B_Amphenol_10103594-0001LF_Horizontal -> VS-TIPI-kicad:AMPHENOL_10118194-0001LF; symbol Connector:USB_B_Micro -> vs-tipi:10118194-0001LF; LCSC (none) -> C132563
- Q1: LCSC (none) -> C31776
- R1, R3: LCSC (none) -> C17513
- R2: LCSC (none) -> C17630
- R4, R5: LCSC (none) -> C17414
- U1: LCSC (none) -> C45126
- U3: LCSC (none) -> C5980
- U4: LCSC (none) -> C23984
- U5: value CY62256L-70PC -> AS6C62256-55PCN
Connections:
- net +5V: now also J3.1 (Pin_1)
- net GND: now also J2.S1 (SHIELD), J2.S2 (SHIELD), J2.S3 (SHIELD), J2.S4 (SHIELD), J2.S5 (SHIELD), J2.S6 (SHIELD), J3.2 (Pin_2); no longer J2.6 (Shield)
Other:
- moved on the sheet: C1, C2, U4
