File: hardware/tipi-peb/kicad/tipi-peb.sch (KiCad schematic (older format))
At the start: 47 parts, among them J1 GS3, J2 GS3, Q1 Q_NPN_BCE, U1 74HCT138, U2 27C256, U3 74HCT244, U4 74HCT244, U5 74HCT244, U6 XC95144XL-TQ100, U7 74HCT245, U8 LM1117-3.3, U9 LM7805_TO220

Commit message: looks ok in latest kicad, but some footprint complaints when 'checking' the board.
Parts:
- C1, C10, C11, C12, C13, C2, C3, C4, C5, C6, C7, C8, C9: symbol tipi-peb-rescue:C_Small -> tipi-peb-rescue:C_Small-tipi-peb-rescue
- C14, C15, C16, C17: symbol tipi-peb-rescue:CP1_Small -> tipi-peb-rescue:CP1_Small-tipi-peb-rescue
- CRUBASE1: symbol tipi-peb-rescue:Conn_02x04_Counter_Clockwise -> tipi-peb-rescue:Conn_02x04_Counter_Clockwise-tipi-peb-rescue
- D1: symbol tipi-peb-rescue:LED_ALT -> tipi-peb-rescue:LED_ALT-tipi-peb-rescue
- J1, J2: symbol tipi-peb-rescue:GS3 -> tipi-peb-rescue:GS3-tipi-peb-rescue
- JTAG1: symbol tipi-peb-rescue:AVR-JTAG-10 -> tipi-peb-rescue:AVR-JTAG-10-tipi-peb-rescue
- Q1: symbol tipi-peb-rescue:Q_NPN_BCE -> tipi-peb-rescue:Q_NPN_BCE-tipi-peb-rescue
- R1, R10, R11, R12, R13, R2, R3, R4, R5, R6: symbol tipi-peb-rescue:R -> tipi-peb-rescue:R-tipi-peb-rescue
- R7, R8, R9: symbol tipi-peb-rescue:R_Small -> tipi-peb-rescue:R_Small-tipi-peb-rescue
- RPi1: symbol tipi-peb-rescue:Conn_02x05_Counter_Clockwise -> tipi-peb-rescue:Conn_02x05_Counter_Clockwise-tipi-peb-rescue
- U1: symbol tipi-peb-rescue:74LS138 -> tipi-peb-rescue:74LS138-tipi-peb-rescue
- U2: symbol tipi-peb-rescue:27C256 -> tipi-peb-rescue:27C256-tipi-peb-rescue
- U3, U4, U5: symbol tipi-peb-rescue:74HC244 -> tipi-peb-rescue:74HC244-tipi-peb-rescue
- U6: symbol tipi-peb-rescue:XC95144XL-TQ100 -> tipi-peb-rescue:XC95144XL-TQ100-tipi-peb-rescue
- U7: symbol tipi-peb-rescue:74LS245 -> tipi-peb-rescue:74LS245-tipi-peb-rescue
- U8: symbol tipi-peb-rescue:LM1117-3.3 -> tipi-peb-rescue:LM1117-3.3-tipi-peb-rescue
- U9: symbol tipi-peb-rescue:LM7805_TO220 -> tipi-peb-rescue:LM7805_TO220-tipi-peb-rescue
Changed lines of the file:
@@
 EESchema Schematic File Version 4
-LIBS:tipi-peb-cache
-EELAYER 26 0
+EELAYER 30 0
 EELAYER END
 $Descr B 17000 11000
@@
 $EndComp
 $Comp
-L tipi-peb-rescue:27C256 U2
+L tipi-peb-rescue:27C256-tipi-peb-rescue U2
 U 1 1 5917F7B0
 P 2050 2100
@@
 $EndComp
 $Comp
-L tipi-peb-rescue:74LS245 U7
+L tipi-peb-rescue:74LS245-tipi-peb-rescue U7
 U 1 1 5917F86D
 P 10250 9400
@@
 $EndComp
 $Comp
-L tipi-peb-rescue:C_Small C9
+L tipi-peb-rescue:C_Small-tipi-peb-rescue C9
 U 1 1 5917FDFE
 P 8500 850
@@
 JTAG_TMS
 $Comp
-L tipi-peb-rescue:AVR-JTAG-10 JTAG1
+L tipi-peb-rescue:AVR-JTAG-10-tipi-peb-rescue JTAG1
 U 1 1 591AA716
 P 14650 1500
@@
 TI_CRUIN
 $Comp
-L tipi-peb-rescue:LM1117-3.3 U8
+L tipi-peb-rescue:LM1117-3.3-tipi-peb-rescue U8
 U 1 1 594EAE75
 P 14450 4250
@@
 $EndComp
 $Comp
-L tipi-peb-rescue:CP1_Small C16
+L tipi-peb-rescue:CP1_Small-tipi-peb-rescue C16
 U 1 1 594EB02A
 P 14850 4350
@@
 $EndComp
 $Comp
-L tipi-peb-rescue:CP1_Small C14
+L tipi-peb-rescue:CP1_Small-tipi-peb-rescue C14
 U 1 1 594EB077
 P 14050 4350
@@
 $EndComp
 $Comp
-L tipi-peb-rescue:LED_ALT D1
+L tipi-peb-rescue:LED_ALT-tipi-peb-rescue D1
 U 1 1 594FDAB3
 P 12350 1200
@@
 $EndComp
 $Comp
-L tipi-peb-rescue:R R6
+L tipi-peb-rescue:R-tipi-peb-rescue R6
 U 1 1 594FDB4A
 P 12750 1200
@@
 $EndComp
 $Comp
-L tipi-peb-rescue:R R5
+L tipi-peb-rescue:R-tipi-peb-rescue R5
 U 1 1 594FDDEA
 P 11650 900
@@
 $EndComp
 $Comp
-L tipi-peb-rescue:Q_NPN_BCE Q1
+L tipi-peb-rescue:Q_NPN_BCE-tipi-peb-rescue Q1
 U 1 1 594FDE57
 P 11900 1100
@@
 LED0
 $Comp
-L tipi-peb-rescue:Conn_02x04_Counter_Clockwise CRUBASE1
+L tipi-peb-rescue:Conn_02x04_Counter_Clockwise-tipi-peb-rescue CRUBASE1
 U 1 1 594FE925
 P 11800 2350
@@
 $EndComp
 $Comp
-L tipi-peb-rescue:Conn_02x05_Counter_Clockwise RPi1
+L tipi-peb-rescue:Conn_02x05_Counter_Clockwise-tipi-peb-rescue RPi1
 U 1 1 594FFC97
 P 14350 3000
@@
 NoConn ~ 14450 1600
 $Comp
-L tipi-peb-rescue:C_Small C2
+L tipi-peb-rescue:C_Small-tipi-peb-rescue C2
 U 1 1 59595B0D
 P 2250 1000
@@
 $EndComp
 $Comp
-L tipi-peb-rescue:C_Small C13
+L tipi-peb-rescue:C_Small-tipi-peb-rescue C13
 U 1 1 595963F1
 P 10400 8550
@@
 $EndComp
 $Comp
-L tipi-peb-rescue:R_Small R7
+L tipi-peb-rescue:R_Small-tipi-peb-rescue R7
 U 1 1 59612E43
 P 13900 2050
@@
 $EndComp
 $Comp
-L tipi-peb-rescue:R_Small R8
+L tipi-peb-rescue:R_Small-tipi-peb-rescue R8
 U 1 1 59612F26
 P 14100 2050
@@
 $EndComp
 $Comp
-L tipi-peb-rescue:R_Small R9
+L tipi-peb-rescue:R_Small-tipi-peb-rescue R9
 U 1 1 59612F85
 P 14300 2050
@@
 $EndComp
 $Comp
-L tipi-peb-rescue:C_Small C10
+L tipi-peb-rescue:C_Small-tipi-peb-rescue C10
 U 1 1 596F064F
 P 8750 850
@@
 $EndComp
 $Comp
-L tipi-peb-rescue:C_Small C11
+L tipi-peb-rescue:C_Small-tipi-peb-rescue C11
 U 1 1 596F06B9
 P 9000 850
@@
 $EndComp
 $Comp
-L tipi-peb-rescue:C_Small C12
+L tipi-peb-rescue:C_Small-tipi-peb-rescue C12
 U 1 1 596F06CB
 P 9250 850
@@
 $EndComp
 $Comp
-L tipi-peb-rescue:C_Small C7
+L tipi-peb-rescue:C_Small-tipi-peb-rescue C7
 U 1 1 596F0DF9
 P 8250 850
@@
 $EndComp
 $Comp
-L tipi-peb-rescue:C_Small C6
+L tipi-peb-rescue:C_Small-tipi-peb-rescue C6
 U 1 1 596F0E6D
 P 8000 850
@@
 $EndComp
 $Comp
-L tipi-peb-rescue:C_Small C5
+L tipi-peb-rescue:C_Small-tipi-peb-rescue C5
 U 1 1 596F0E7F
 P 7750 850
@@
 $EndComp
 $Comp
-L tipi-peb-rescue:XC95144XL-TQ100 U6
+L tipi-peb-rescue:XC95144XL-TQ100-tipi-peb-rescue U6
 U 1 1 596EEAA9
 P 8550 4100
@@
 $EndComp
 $Comp
-L tipi-peb-rescue:R R4
+L tipi-peb-rescue:R-tipi-peb-rescue R4
 U 1 1 599E6C64
 P 11450 2300
@@
 TI_D7
 $Comp
-L tipi-peb-rescue:74HC244 U5
+L tipi-peb-rescue:74HC244-tipi-peb-rescue U5
 U 1 1 59C69B40
 P 8150 9400
@@
 $EndComp
 $Comp
-L tipi-peb-rescue:74HC244 U4
+L tipi-peb-rescue:74HC244-tipi-peb-rescue U4
 U 1 1 59C69BE6
 P 5800 9400
@@
 $EndComp
 $Comp
-L tipi-peb-rescue:74HC244 U3
+L tipi-peb-rescue:74HC244-tipi-peb-rescue U3
 U 1 1 59C69C7A
 P 3750 9400
@@
 $EndComp
 $Comp
-L tipi-peb-rescue:R R2
+L tipi-peb-rescue:R-tipi-peb-rescue R2
 U 1 1 59C6B529
 P 5350 10050
@@
 $EndComp
 $Comp
-L tipi-peb-rescue:R R3
+L tipi-peb-rescue:R-tipi-peb-rescue R3
 U 1 1 59C6B916
 P 7700 10050
@@
 $EndComp
 $Comp
-L tipi-peb-rescue:R R1
+L tipi-peb-rescue:R-tipi-peb-rescue R1
 U 1 1 59C6CE84
 P 3300 10100
@@
 TI_WE
 $Comp
-L tipi-peb-rescue:74LS138 U1
+L tipi-peb-rescue:74LS138-tipi-peb-rescue U1
 U 1 1 59C72E85
 P 1850 9300
@@
 	3150 9600 3150 9800
 $Comp
-L tipi-peb-rescue:C_Small C1
+L tipi-peb-rescue:C_Small-tipi-peb-rescue C1
 U 1 1 59C76A23
 P 2000 8550
@@
 Connection ~ 1850 8650
 $Comp
-L tipi-peb-rescue:C_Small C3
+L tipi-peb-rescue:C_Small-tipi-peb-rescue C3
 U 1 1 59C76B96
 P 3900 8500
@@
 	3750 8600 3750 8700
 $Comp
-L tipi-peb-rescue:C_Small C4
+L tipi-peb-rescue:C_Small-tipi-peb-rescue C4
 U 1 1 59C76D70
 P 5950 8500
@@
 	5800 8600 5800 8700
 $Comp
-L tipi-peb-rescue:C_Small C8
+L tipi-peb-rescue:C_Small-tipi-peb-rescue C8
 U 1 1 59C76E70
 P 8300 8500
@@
 $EndComp
 $Comp
-L tipi-peb-rescue:LM7805_TO220 U9
+L tipi-peb-rescue:LM7805_TO220-tipi-peb-rescue U9
 U 1 1 59E1BD59
 P 14450 5200
@@
 $EndComp
 $Comp
-L tipi-peb-rescue:CP1_Small C15
+L tipi-peb-rescue:CP1_Small-tipi-peb-rescue C15
 U 1 1 59E1BE91
 P 14050 5300
@@
 $EndComp
 $Comp
-L tipi-peb-rescue:CP1_Small C17
+L tipi-peb-rescue:CP1_Small-tipi-peb-rescue C17
 U 1 1 59E1BF3C
 P 14850 5300
@@
 Connection ~ 3150 9800
 $Comp
-L tipi-peb-rescue:R R10
+L tipi-peb-rescue:R-tipi-peb-rescue R10
 U 1 1 59EF200E
 P 850 8100
@@
 $EndComp
 $Comp
-L tipi-peb-rescue:R R11
+L tipi-peb-rescue:R-tipi-peb-rescue R11
 U 1 1 59EF20E5
 P 1200 7850
@@
 	1000 9650 1250 9650
 $Comp
-L tipi-peb-rescue:R R12
+L tipi-peb-rescue:R-tipi-peb-rescue R12
 U 1 1 5ADB77AD
 P 2900 9400
@@
 Connection ~ 15000 3100
 $Comp
-L tipi-peb-rescue:R R13
+L tipi-peb-rescue:R-tipi-peb-rescue R13
 U 1 1 5B0C3DBA
 P 15000 3500
@@
 	15000 3650 15150 3650
 $Comp
-L tipi-peb-rescue:GS3 J1
+L tipi-peb-rescue:GS3-tipi-peb-rescue J1
 U 1 1 5B12C05D
 P 750 8600
@@
 $EndComp
 $Comp
-L tipi-peb-rescue:GS3 J2
+L tipi-peb-rescue:GS3-tipi-peb-rescue J2
 U 1 1 5B12C0F2
 P 1100 8300
