File: hardware/tipi-peb/kicad/tipi-peb.kicad_pcb (KiCad board)
At the start: 2 copper layers, 237.7 x 146.1 mm, 51 parts, among them J1 GS3, J2 GS3, Q1 Q_NPN_BCE, U1 74HCT138, U2 27C256, U3 74HCT244, U4 74HCT244, U5 74HCT244, U6 XC95144XL-TQ100, U7 74HCT245, U8 LM1117-3.3, U9 LM7805_TO220

Commit message: magic conversion to kicad 6
Other:
- net class Default removed
